Commit message: Add LiDAR, room world, ground truth and switchable odometry to the sim
- gpu_lidar modelled on the YDLIDAR X4 Pro (/scan, 720 samples, 7 Hz)
- room.sdf: 5x4 m room with furniture, now the default world
- /ground_truth/odom from the OdometryPublisher system
- odom_source:=gazebo|user: user mode leaves /odom and odom->base_footprint
  to your own node and moves the plugin estimate to /diff_drive/odom
- joint_state_throttle republishes /joint_states at a fixed rate
  (Fortress publishes every physics step)
- RViz config (rviz:=true) and DISPLAY fallback for headless LiDAR rendering

Co-Authored-By: Claude Opus 5.5 <noreply@anthropic.com>

File: roomba_gazebo/urdf/roomba.urdf.xacro (robot description, xacro)
@@ -117,4 +117,64 @@
   <xacro:caster prefix="front" x="${caster_x}"/>
   <xacro:caster prefix="rear" x="${-caster_x}"/>
+  <!-- YDLIDAR X4 Pro: 360 deg, 0.12-10 m, ~5k samples/s. Mount pose is a placeholder
+       until the 3D-printed mount exists; measure it and update these. -->
+  <xacro:property name="laser_x" value="0.0"/>
+  <xacro:property name="laser_z" value="0.11"/>
+  <xacro:property name="laser_rate" value="7"/>
+  <xacro:property name="laser_samples" value="720"/>
+  <link name="laser_link">
+    <inertial>
+      <mass value="0.18"/>
+      <inertia ixx="1e-4" ixy="0" ixz="0" iyy="1e-4" iyz="0" izz="1e-4"/>
+    </inertial>
+    <visual>
+      <origin xyz="0 0 -0.017"/>
+      <geometry>
+        <cylinder radius="0.035" length="0.034"/>
+      </geometry>
+    </visual>
+    <collision>
+      <origin xyz="0 0 -0.017"/>
+      <geometry>
+        <cylinder radius="0.035" length="0.034"/>
+      </geometry>
+    </collision>
+  </link>
+  <joint name="laser_joint" type="fixed">
+    <origin xyz="${laser_x} 0 ${laser_z - base_z}"/>
+    <parent link="base_link"/>
+    <child link="laser_link"/>
+  </joint>
+  <gazebo reference="laser_link">
+    <sensor name="lidar" type="gpu_lidar">
+      <ignition_frame_id>laser_link</ignition_frame_id>
+      <topic>/scan</topic>
+      <update_rate>${laser_rate}</update_rate>
+      <always_on>true</always_on>
+      <visualize>false</visualize>
+      <lidar>
+        <scan>
+          <horizontal>
+            <samples>${laser_samples}</samples>
+            <resolution>1</resolution>
+            <min_angle>${-PI}</min_angle>
+            <max_angle>${PI - 2 * PI / laser_samples}</max_angle>
+          </horizontal>
+        </scan>
+        <range>
+          <min>0.12</min>
+          <max>10.0</max>
+          <resolution>0.01</resolution>
+        </range>
+        <noise>
+          <type>gaussian</type>
+          <mean>0.0</mean>
+          <stddev>0.01</stddev>
+        </noise>
+      </lidar>
+    </sensor>
+  </gazebo>
+  <!-- Gazebo-side topics live under /diff_drive and /ground_truth; the launch file's
+       bridge decides which of them become /odom and /tf on the ROS side. -->
   <gazebo>
     <plugin filename="ignition-gazebo-diff-drive-system"
@@ -127,9 +187,20 @@
       <max_linear_velocity>0.5</max_linear_velocity>
       <topic>/cmd_vel</topic>
-      <odom_topic>/odom</odom_topic>
-      <tf_topic>/tf</tf_topic>
+      <odom_topic>/diff_drive/odom</odom_topic>
+      <tf_topic>/diff_drive/tf</tf_topic>
       <frame_id>odom</frame_id>
       <child_frame_id>base_footprint</child_frame_id>
       <odom_publish_frequency>50</odom_publish_frequency>
+    </plugin>
+    <!-- True pose from the physics engine, for judging odometry error. The robot is
+         spawned at the world origin, so this is also relative to the start pose. -->
+    <plugin filename="ignition-gazebo-odometry-publisher-system"
+            name="ignition::gazebo::systems::OdometryPublisher">
+      <odom_frame>odom</odom_frame>
+      <robot_base_frame>base_footprint</robot_base_frame>
+      <odom_topic>/ground_truth/odom</odom_topic>
+      <tf_topic>/ground_truth/tf</tf_topic>
+      <odom_publish_frequency>50</odom_publish_frequency>
+      <dimensions>2</dimensions>
     </plugin>
     <plugin filename="ignition-gazebo-joint-state-publisher-system"
